File: examples/rf-coupons/JLC06161H-2116C/board-B.kicad_pcb (KiCad board)
At the start: 6 copper layers, 224 x 120 mm, 90 parts, among them X1 TestPoint_PTH, X10 TestPoint_PTH, X11 TestPoint_PTH, X12 TestPoint_PTH, X13 TestPoint_PTH, X14 TestPoint_PTH, X15 TestPoint_PTH, X16 TestPoint_PTH, X17 TestPoint_PTH, X18 TestPoint_PTH, X19 TestPoint_PTH, X2 TestPoint_PTH, X20 TestPoint_PTH, X21 TestPoint_PTH, X22 TestPoint_PTH, X23 TestPoint_PTH, X24 TestPoint_PTH, X25 TestPoint_PTH, X26 TestPoint_PTH, X27 TestPoint_PTH, X28 TestPoint_PTH, X29 TestPoint_PTH, X3 TestPoint_PTH, X30 TestPoint_PTH, X31 TestPoint_PTH, X32 TestPoint_PTH, X33 TestPoint_PTH, X34 TestPoint_PTH, X35 TestPoint_PTH, X36 TestPoint_PTH, X37 TestPoint_PTH, X38 TestPoint_PTH, X39 TestPoint_PTH, X4 TestPoint_PTH, X40 TestPoint_PTH, X41 TestPoint_PTH, X42 TestPoint_PTH, X43 TestPoint_PTH, X44 TestPoint_PTH, X45 TestPoint_PTH, X46 TestPoint_PTH, X47 TestPoint_PTH, X48 TestPoint_PTH, X49 TestPoint_PTH, X5 TestPoint_PTH, X50 TestPoint_PTH, X51 TestPoint_PTH, X52 TestPoint_PTH, X57 Microsection, X58 Anchor, X6 TestPoint_PTH, X7 TestPoint_PTH, X8 TestPoint_PTH, X9 TestPoint_PTH

Commit message: Order 0: the uploads and predictions regenerated after the review
examples/rf-coupons/order0: generated from 73fe6527 (the tag carries it); KiCad
DRC under OSH Park's 4-layer rules 0 violations / 0 unconnected on all three.
`yapnr fab check` (oshpark-4l, oshpark-4l-fr408hr): O0-M 0 errors; O0-W and
O0-D stop on FAB-PLACEHOLDER until D2 and D1 are in (by design); warnings as
before (NPTH in the merged drill file; 1.511 mm of published layers):

- O0-M 120.1 x 144.3 mm, 26.9 sq in, 33 SMAs per copy, 32 tabs;
- O0-W 57.5 x 131.2 mm, 11.7 sq in, 16 SMAs, 15 tabs;
- O0-D 90.6 x 51.5 mm, 7.2 sq in, 12 SMAs, 9 tabs (A20 added).

Every stick has two or more tabs, all on edges without a launch; no plane via
under a silkscreen glyph; no mask web under 0.1 mm; the QR decodes from the
silkscreen render.

Predictions: the coupons on FR408HR and EM528 with the review's roughness
prior, the junction-corrected ring and stub (A12 notch 5.500 GHz FR408HR,
5.388 GHz EM528; A11 1.924 / 5.793 GHz), scalars.json and lines.csv. Boards A
and B regenerated (mask-opening anchors only; DRC unchanged).

docs/rf/order0: sizes and costs, R1/R1t as drawn, the renormalization to the
solver's port impedance (review H3), the C-pad method (M3), the loss basis
(M4), the scalars (L1), the sha256 rule (F9), the connector-fit pre-check, the
mask web note (L2), and the D1/D2 pages with the board around each window.

Co-Authored-By: Claude Opus 5.5 <noreply@anthropic.com>
Claude-Session: https://claude.ai/code/session_01NY8rMuBH8hTFjkoZyuqNZ7
Parts:
- moved MO_B24 20.1 mm to (161.0, 101.6)
Changed lines of the file:
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@@
 		(fp_rect (start -2.35 -3.75) (end 2.1 3.75) (stroke (width 0.05) (type solid)) (fill no) (layer "F.CrtYd"))
 	)
-	(footprint "MaskOpening" (layer "F.Cu") (at 181 103.5 0)
+	(footprint "MaskOpening" (layer "F.Cu") (at 161 101.62 0)
 		(property "Reference" "MO_B24" (at 0 0 0) (layer "F.Fab") (effects (font (size 0.8 0.8) (thickness 0.12))))
 		(property "Value" "MaskOpening" (at 0 0 0) (layer "F.Fab") (hide yes) (effects (font (size 0.8 0.8) (thickness 0.12))))
 		(attr smd)
-		(fp_poly (pts (xy -20 -1.875) (xy 20 -1.875) (xy 20 1.875) (xy -20 1.875)) (stroke (width 0) (type solid)) (fill yes) (layer "F.Mask"))
+		(fp_poly (pts (xy 0 0.005) (xy 40 0.005) (xy 40 3.755) (xy 0 3.755)) (stroke (width 0) (type solid)) (fill yes) (layer "F.Mask"))
 	)
 	(footprint "SMA_EdgeLaunch_SMA-J-P-H-ST-EM1" (layer "F.Cu") (at 215.1 103.5 180)
