File: examples/radar60/board/radar60.kicad_pcb (KiCad board)
At the start: 6 copper layers, 60 x 47.3 mm, 6 parts

Commit message: radar60 board: stage 3b floorplan (regions, exit-band slots, anchored groups, fanout)
floorplan.yaml (and the generated constraints.yaml and floorplan board):

- J2 and J3 are region parts again (x 8-34, y 7.25-15.6; x 0.6-8.3, y 8-24.3):
  J2's fixed stage-2 pose predates the QTH land and the 47.35 mm board;
- Y1 moves east of the SPIA exit band and below its load caps (x 28.4-33.0,
  y 15.75-19.7); the CLKM cap stands upright over C15's band, the CLKP cap flat
  east of it (pads 2.0 and 2.5 mm from their balls); the QSPI clock resistor
  sits just west of the R12 neighbours' bands (about 4.5 mm from R12);
- pad-anchored hard groups: each snubber resistor within 3.5 mm of its
  inductor's switch-node pad (replacing 7.5 mm from U2's centre), the 1V0_RF1
  ferrite within 12 mm of H5, the 1V0_RF2 ferrites within 10 mm of D2, each DNP
  damping resistor within 3 mm of its ferrite's rail pad and its capacitor within
  2 mm of the resistor;
- copper_keepout v1 replaces the U1-frame v0 rectangles that forbade the macro's
  own copper: the RF region (macro group exempt), the R4 guard (RF, PWR, GND,
  ANALOG allowed), the mounting-hole and radome-land circles, and no via under
  the flash's exposed pad (Macronix);
- fixed_block rfm1 (group RFM1_MACRO, anchored at U1, In2 GND solid), U1's
  fanout (trial 2's entry; A2/B2 skipped until macro v2 owns the VOUT_PA feed,
  D14; six bottom sites), plane_fallback_drops false, and the legalizer options
  outline exact, order scarcity, lookahead regions.

The README's floorplan table follows the 47.35 mm board and the new inputs.

Co-Authored-By: Claude Opus 5.5 <noreply@anthropic.com>
Claude-Session: https://claude.ai/code/session_014FiHUDEn5jCP4V8pPjQkPy
Other:
- board text added: "jtag"
- board text added: "lvds_header"
Changed lines of the file:
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@@
 	(zone (net 0) (net_name "") (layers "F.Cu" "In1.Cu" "In2.Cu" "In3.Cu" "In4.Cu" "B.Cu") (name "RADOME_LAND1_KEEPOUT") (hatch edge 0.5) (connect_pads (clearance 0)) (min_thickness 0.25) (filled_areas_thickness no) (keepout (tracks not_allowed) (vias not_allowed) (pads allowed) (copperpour allowed) (footprints allowed)) (placement (enabled no) (sheetname "")) (fill (thermal_gap 0.5) (thermal_bridge_width 0.5)) (polygon (pts (xy 36 50.35) (xy 35.9148 49.703) (xy 35.6651 49.1) (xy 35.2678 48.5822) (xy 34.75 48.1849) (xy 34.147 47.9352) (xy 33.5 47.85) (xy 32.853 47.9352) (xy 32.25 48.1849) (xy 31.7322 48.5822) (xy 31.3349 49.1) (xy 31.0852 49.703) (xy 31 50.35) (xy 31.0852 50.997) (xy 31.3349 51.6) (xy 31.7322 52.1178) (xy 32.25 52.5151) (xy 32.853 52.7648) (xy 33.5 52.85) (xy 34.147 52.7648) (xy 34.75 52.5151) (xy 35.2678 52.1178) (xy 35.6651 51.6) (xy 35.9148 50.997))))
 	(zone (net 0) (net_name "") (layers "F.Cu" "In1.Cu" "In2.Cu" "In3.Cu" "In4.Cu" "B.Cu") (name "RADOME_LAND2_KEEPOUT") (hatch edge 0.5) (connect_pads (clearance 0)) (min_thickness 0.25) (filled_areas_thickness no) (keepout (tracks not_allowed) (vias not_allowed) (pads allowed) (copperpour allowed) (footprints allowed)) (placement (enabled no) (sheetname "")) (fill (thermal_gap 0.5) (thermal_bridge_width 0.5)) (polygon (pts (xy 89 50.35) (xy 88.9148 49.703) (xy 88.6651 49.1) (xy 88.2678 48.5822) (xy 87.75 48.1849) (xy 87.147 47.9352) (xy 86.5 47.85) (xy 85.853 47.9352) (xy 85.25 48.1849) (xy 84.7322 48.5822) (xy 84.3349 49.1) (xy 84.0852 49.703) (xy 84 50.35) (xy 84.0852 50.997) (xy 84.3349 51.6) (xy 84.7322 52.1178) (xy 85.25 52.5151) (xy 85.853 52.7648) (xy 86.5 52.85) (xy 87.147 52.7648) (xy 87.75 52.5151) (xy 88.2678 52.1178) (xy 88.6651 51.6) (xy 88.9148 50.997))))
+	(gr_rect (start 38 61.75) (end 64 70.1) (stroke (width 0.1) (type dash)) (fill no) (layer "User.1"))
+	(gr_text "lvds_header" (at 38.3 62.65 0) (layer "User.1") (effects (font (size 0.6 0.6) (thickness 0.12)) (justify left)))
+	(gr_rect (start 30.6 53.05) (end 38.3 69.35) (stroke (width 0.1) (type dash)) (fill no) (layer "User.1"))
+	(gr_text "jtag" (at 30.9 53.95 0) (layer "User.1") (effects (font (size 0.6 0.6) (thickness 0.12)) (justify left)))
 	(gr_rect (start 68 50.7) (end 88 75.35) (stroke (width 0.1) (type dash)) (fill no) (layer "User.1"))
 	(gr_text "pmic_block" (at 68.3 51.6 0) (layer "User.1") (effects (font (size 0.6 0.6) (thickness 0.12)) (justify left)))
@@
 	(gr_rect (start 71 55.65) (end 88 75.35) (stroke (width 0.1) (type dash)) (fill no) (layer "User.1"))
 	(gr_text "pmic_switching" (at 71.3 56.55 0) (layer "User.1") (effects (font (size 0.6 0.6) (thickness 0.12)) (justify left)))
-	(gr_rect (start 53.5 55.8) (end 60.2 61.6) (stroke (width 0.1) (type dash)) (fill no) (layer "User.1"))
-	(gr_text "crystal" (at 53.8 56.7 0) (layer "User.1") (effects (font (size 0.6 0.6) (thickness 0.12)) (justify left)))
+	(gr_rect (start 58.4 57.65) (end 63 61.6) (stroke (width 0.1) (type dash)) (fill no) (layer "User.1"))
+	(gr_text "crystal" (at 58.7 58.55 0) (layer "User.1") (effects (font (size 0.6 0.6) (thickness 0.12)) (justify left)))
 	(gr_rect (start 62.1 50.9) (end 64.15 52.05) (stroke (width 0.1) (type dash)) (fill no) (layer "User.1"))
 	(gr_text "radio_apll" (at 62.4 51.8 0) (layer "User.1") (effects (font (size 0.6 0.6) (thickness 0.12)) (justify left)))
@@
 	(gr_rect (start 62.1 53.4) (end 64.15 54.55) (stroke (width 0.1) (type dash)) (fill no) (layer "User.1"))
 	(gr_text "radio_synth" (at 62.4 54.3 0) (layer "User.1") (effects (font (size 0.6 0.6) (thickness 0.12)) (justify left)))
-	(gr_rect (start 59.1 55.4) (end 61.15 56.55) (stroke (width 0.1) (type dash)) (fill no) (layer "User.1"))
-	(gr_text "xtal_cap_p" (at 59.4 56.3 0) (layer "User.1") (effects (font (size 0.6 0.6) (thickness 0.12)) (justify left)))
-	(gr_rect (start 56.85 55.4) (end 58.9 56.55) (stroke (width 0.1) (type dash)) (fill no) (layer "User.1"))
-	(gr_text "xtal_cap_n" (at 57.15 56.3 0) (layer "User.1") (effects (font (size 0.6 0.6) (thickness 0.12)) (justify left)))
+	(gr_rect (start 59.5 55.65) (end 61.7 57.05) (stroke (width 0.1) (type dash)) (fill no) (layer "User.1"))
+	(gr_text "xtal_cap_p" (at 59.8 56.55 0) (layer "User.1") (effects (font (size 0.6 0.6) (thickness 0.12)) (justify left)))
+	(gr_rect (start 58.2 55.3) (end 59.6 57.45) (stroke (width 0.1) (type dash)) (fill no) (layer "User.1"))
+	(gr_text "xtal_cap_n" (at 58.5 56.2 0) (layer "User.1") (effects (font (size 0.6 0.6) (thickness 0.12)) (justify left)))
 	(gr_rect (start 60.05 45.5) (end 61.2 47.95) (stroke (width 0.1) (type dash)) (fill no) (layer "User.1"))
 	(gr_text "pa_cap" (at 60.35 46.4 0) (layer "User.1") (effects (font (size 0.6 0.6) (thickness 0.12)) (justify left)))
@@
 	(gr_rect (start 45 44.35) (end 49.55 51.35) (stroke (width 0.1) (type dash)) (fill no) (layer "User.1"))
 	(gr_text "radio_west" (at 45.3 45.25 0) (layer "User.1") (effects (font (size 0.6 0.6) (thickness 0.12)) (justify left)))
-	(gr_rect (start 47.85 51.4) (end 49.95 52.55) (stroke (width 0.1) (type dash)) (fill no) (layer "User.1"))
-	(gr_text "qspi_series" (at 48.15 52.3 0) (layer "User.1") (effects (font (size 0.6 0.6) (thickness 0.12)) (justify left)))
+	(gr_rect (start 45.4 51.4) (end 47.55 52.55) (stroke (width 0.1) (type dash)) (fill no) (layer "User.1"))
+	(gr_text "qspi_series" (at 45.7 52.3 0) (layer "User.1") (effects (font (size 0.6 0.6) (thickness 0.12)) (justify left)))
 	(gr_rect (start 61.6 66.35) (end 68.5 70.7) (stroke (width 0.1) (type dash)) (fill no) (layer "User.1"))
 	(gr_text "connector_esd" (at 61.9 67.25 0) (layer "User.1") (effects (font (size 0.6 0.6) (thickness 0.12)) (justify left)))
