File: examples/radar60/board/radar60.kicad_pcb (KiCad board)
At the start: 6 copper layers, 60 x 47.3 mm, 6 parts

Commit message: radar60 R1: the power stage as two subcells (U2 buck stage, U5 eFuse stage)
One rigid block holding U2's and U5's clusters (37 parts, 450-715 mm2 synthesized)
fitted no legal place in 24 of 24 hierarchical top starts (wave 4: "MB00 fits nowhere ...
region pmic_block" / "no free slot"): the pmic regions are 20 mm wide and the strip west
of J1 under J2 is 6.55 mm tall. The subcell splits along its own hard-group clusters:

- floorplan power_stage.blocks: the buck stage at U2 (inductors, input caps, snubbers,
  VANA, R_SH1, TP1; F.Cu pours for 5V_SYS, SW_B0-3, 1V0_BUCK, GND) and the eFuse stage
  at U5 (D3, C33/C34 in, C36/C37 out; pours for VIN_5V, 5V_SYS, GND), each with its own
  fixed_block, hot loops and outline grid; efuse_block/connector_tvs regions restored;
  the eFuse threshold group is soft (hard: false, gen_board passes it), since a hard group
  may not straddle a rigid block and the 11 parts do not fit the strip with U5.
- power_block.py: --block-anchor picks the block; merge joins the libraries.

Co-Authored-By: Claude Opus 5.5 <noreply@anthropic.com>
Claude-Session: https://claude.ai/code/session_01XmUgXgxLjzBpn2W6JpqE2p
Other:
- board text added: "connector_tvs"
- board text added: "efuse_block"
Changed lines of the file:
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@@
 	(gr_rect (start 38.3 52.75) (end 49.3 61.6) (stroke (width 0.1) (type dash)) (fill no) (layer "User.1"))
 	(gr_text "flash_block" (at 38.6 53.65 0) (layer "User.1") (effects (font (size 0.6 0.6) (thickness 0.12)) (justify left)))
+	(gr_rect (start 36.8 70.1) (end 52.5 76.95) (stroke (width 0.1) (type dash)) (fill no) (layer "User.1"))
+	(gr_text "efuse_block" (at 37.1 71 0) (layer "User.1") (effects (font (size 0.6 0.6) (thickness 0.12)) (justify left)))
 	(gr_rect (start 61.6 61.35) (end 68 70.7) (stroke (width 0.1) (type dash)) (fill no) (layer "User.1"))
 	(gr_text "can_block" (at 61.9 62.25 0) (layer "User.1") (effects (font (size 0.6 0.6) (thickness 0.12)) (justify left)))
@@
 	(gr_rect (start 61.6 66.35) (end 68.5 70.7) (stroke (width 0.1) (type dash)) (fill no) (layer "User.1"))
 	(gr_text "connector_esd" (at 61.9 67.25 0) (layer "User.1") (effects (font (size 0.6 0.6) (thickness 0.12)) (justify left)))
+	(gr_rect (start 42 70.1) (end 52.5 76.95) (stroke (width 0.1) (type dash)) (fill no) (layer "User.1"))
+	(gr_text "connector_tvs" (at 42.3 71 0) (layer "User.1") (effects (font (size 0.6 0.6) (thickness 0.12)) (justify left)))
 	(gr_rect (start 47.599 35.336) (end 60.759 39.387) (stroke (width 0.1) (type dash)) (fill no) (layer "User.2"))
 	(gr_text "RX patches" (at 47.599 35.036 0) (layer "User.2") (effects (font (size 0.6 0.6) (thickness 0.12)) (justify left)))

Commit message: radar60 floorplan (R1, R3): one power-stage subcell around U2 and U5; In3 partitioned in the plan's order
R1: two hard groups join U2's (inductors, input caps, snubbers, VANA, R_SH1) with U5's
(thresholds, in/out caps) and put D3 at the eFuse input and TP1 at R_SH1, so
pnr.hier.blocks extracts one power-stage block; the eFuse and TVS regions west of J1 go
(a rigid block cannot hold both them and pmic_switching). A new floorplan `power_stage`
section names the block, its fixed_block (PWR_STAGE, anchored on U2, F.Cu solid), the
outer F.Cu pours for the hot-rod lands (region, whole-land terminals, solid connection)
and the datasheet hot loops the synthesis ranks by.

R3: In3 partition nets 1V0_RF1, 1V0_RF2, 1V0_PA, 1V2, 1V8, 5V_SYS, 1V0_SH, order listed,
fixed_lands; 1V0_SH keeps its 0.5 mOhm report but does not widen its trunk (owner Q2
default, local sensing). gen_board.py passes order/fixed_lands/no_budget through.

Co-Authored-By: Claude Opus 5.5 <noreply@anthropic.com>
Claude-Session: https://claude.ai/code/session_01XmUgXgxLjzBpn2W6JpqE2p
Other:
- board text removed: "connector_tvs"
- board text removed: "efuse_block"
Changed lines of the file:
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@@
 	(gr_rect (start 38.3 52.75) (end 49.3 61.6) (stroke (width 0.1) (type dash)) (fill no) (layer "User.1"))
 	(gr_text "flash_block" (at 38.6 53.65 0) (layer "User.1") (effects (font (size 0.6 0.6) (thickness 0.12)) (justify left)))
-	(gr_rect (start 36.8 70.1) (end 52.5 76.95) (stroke (width 0.1) (type dash)) (fill no) (layer "User.1"))
-	(gr_text "efuse_block" (at 37.1 71 0) (layer "User.1") (effects (font (size 0.6 0.6) (thickness 0.12)) (justify left)))
 	(gr_rect (start 61.6 61.35) (end 68 70.7) (stroke (width 0.1) (type dash)) (fill no) (layer "User.1"))
 	(gr_text "can_block" (at 61.9 62.25 0) (layer "User.1") (effects (font (size 0.6 0.6) (thickness 0.12)) (justify left)))
@@
 	(gr_rect (start 61.6 66.35) (end 68.5 70.7) (stroke (width 0.1) (type dash)) (fill no) (layer "User.1"))
 	(gr_text "connector_esd" (at 61.9 67.25 0) (layer "User.1") (effects (font (size 0.6 0.6) (thickness 0.12)) (justify left)))
-	(gr_rect (start 42 70.1) (end 52.5 76.95) (stroke (width 0.1) (type dash)) (fill no) (layer "User.1"))
-	(gr_text "connector_tvs" (at 42.3 71 0) (layer "User.1") (effects (font (size 0.6 0.6) (thickness 0.12)) (justify left)))
 	(gr_rect (start 47.599 35.336) (end 60.759 39.387) (stroke (width 0.1) (type dash)) (fill no) (layer "User.2"))
 	(gr_text "RX patches" (at 47.599 35.036 0) (layer "User.2") (effects (font (size 0.6 0.6) (thickness 0.12)) (justify left)))

Commit message: radar60 re-place (R7, R9): Y1 In2/B.Cu keepout, flash EP F.Cu pour, R46 slot; select --top-n
R9: crystal_keepout bars I2C/CAN/FRAME_START from In2.Cu/B.Cu under Y1 (x 28.9-32.9), allowing
only GND/XTAL; flash_ep.pour adds a local plane_partition region (E1's mechanism) so GND floods
U3's exposed pad instead of relying on a maze track into its own keepout-narrowed courtyard
(wave 1: 0 escape candidates on U3.9).

R7: R46 (radio.r_pa, owner Q1 default WFCP0612 1 mOhm) does not fit its old 0402-sized pa_r
bottom-site slot (2.35 x 1.35 mm vs ~17 mm2 needed) or any area inside U1's BGA shadow. Removed
that region; added a hard group (anchor U1 pad D2, radius 11 mm) so the MC search finds a legal
slot mechanically instead of a hand-picked rect. audit.py's pin-distance PIN_LIMITS split
pa_decoupling's 3 mm hard limit into pa_cap/rf2_cap (unchanged, still fit their slots) and pa_r
(11 mm, soft) -- otherwise every candidate hard-fails on a limit sized for the part R46 no
longer is. The BOM/footprint swap itself is not applied (no atopile here); flagged for the
R2/power-chain track once it is.

gen_board.py: power_sections() and the new flash-EP pour both wrote plane_partition; a dict
merge let the second clobber the first -- fixed to append.

integrate.py: select --top-n writes every legal, audit-passing candidate up to N (ranked) to
candidates/rankN/, not just the stage-0 winner, so a wave can route more than one. New
_top_candidates(), unit-tested (5 cases, hermetic, tests/unit/radar60/test_integrate.py).

Verified: gen_board.py --check/--compile clean; a real source->prepare->place(32 starts) run
through integrate.py (Mac, heavy.sh, KiCad headless) raises no slot/legalization/audit failure
naming R46, Y1, the crystal caps or U3 on any of the 32 starts. 2/32 are legal; both fail the
audit on a J1 VIN_5V protection-order check unrelated to this change (traced to the concurrent
power track's R1 commit re-anchoring connector_tvs off J1; see stage3c/r2-place.md) -- 0/32
write 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
Other:
- board text removed: "pa_r"
Changed lines of the file:
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@@
 	(gr_rect (start 60.05 45.5) (end 61.2 47.95) (stroke (width 0.1) (type dash)) (fill no) (layer "User.1"))
 	(gr_text "pa_cap" (at 60.35 46.4 0) (layer "User.1") (effects (font (size 0.6 0.6) (thickness 0.12)) (justify left)))
-	(gr_rect (start 58.6 44.15) (end 60.95 45.5) (stroke (width 0.1) (type dash)) (fill no) (layer "User.1"))
-	(gr_text "pa_r" (at 58.9 45.05 0) (layer "User.1") (effects (font (size 0.6 0.6) (thickness 0.12)) (justify left)))
 	(gr_rect (start 56.1 44.15) (end 58.6 45.5) (stroke (width 0.1) (type dash)) (fill no) (layer "User.1"))
 	(gr_text "rf2_cap" (at 56.4 45.05 0) (layer "User.1") (effects (font (size 0.6 0.6) (thickness 0.12)) (justify left)))
