File: examples/rf-coupons/order0/O0-W/O0-W.kicad_pcb (KiCad board)
At the start: 4 copper layers, 54 x 158.7 mm, 35 parts, among them X16 Anchor, X18 Anchor

Commit message: Order 0: O0-W review fixes (D2 registration, Gerber hash, docs)
- preregistration.md, predictions/D2/README.md: D2's owner-default text said it passes
  |S21|/|S31| everywhere and misses only |S11| ("measured"). Against the prediction that
  "meets spec" uses (loss-corrected), d2-star-sched's |S21| = |S31| is -3.43 to -3.45 dB on
  W-eq/W-nom, a 0.03-0.05 dB miss of -3.4 dB, and the committed in-job criteria (d2.json,
  -3.40 dB coarse) fail at the coarse grid; it passes only the design's -3.45/-3.6 dB
  validation limits. Both versions reported; "measured" -> predicted; the silkscreen carries
  the hash8 only (run id and DRC status are in catalog.json).
- O0-W board: silkscreen "gen ee9da3f" (the commit whose generator makes this board, B15
  included) instead of ad2bda7; otherwise byte-identical, KiCad DRC 0, fab check 0 errors.
- fab/O0-W.sha256: the Gerber zip to upload (rebuilds reorder flashes, so the release must
  attach this exact zip, as for O0-M); manifest regenerated (also adds BUILD.bazel, missing
  since #53).
- README tables/image: O0-W 54.0 x 158.7 mm, 13.3 sq in, $133, D2 and B15 instead of the
  placeholder; examples README likewise.

Co-Authored-By: Claude Opus 5.5 <noreply@anthropic.com>
Claude-Session: https://claude.ai/code/session_01XmUgXgxLjzBpn2W6JpqE2p
Other:
- board text added: "gen ee9da3f"
- board text removed: "gen ad2bda7"
Changed lines of the file:
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@@
 	(gr_text "yapnr Order 0 rev A O0-W" (at 48.54 93.98 0) (layer "F.SilkS") (effects (font (size 1 1) (thickness 0.15)) (justify left)))
 	(gr_text "oshpark-4l-fr408hr" (at 48.54 95.78 0) (layer "F.SilkS") (effects (font (size 1 1) (thickness 0.15)) (justify left)))
-	(gr_text "gen ad2bda7" (at 48.54 97.58 0) (layer "F.SilkS") (effects (font (size 1 1) (thickness 0.15)) (justify left)))
+	(gr_text "gen ee9da3f" (at 48.54 97.58 0) (layer "F.SilkS") (effects (font (size 1 1) (thickness 0.15)) (justify left)))
 	(gr_line (start 51.54 82.58) (end 54.54 82.58) (stroke (width 0.15) (type solid)) (layer "B.SilkS"))
 	(gr_line (start 54.54 82.58) (end 54.54 85.58) (stroke (width 0.15) (type solid)) (layer "B.SilkS"))
